File: mainv2/mainv2.kicad_sch (KiCad schematic)
At the start: 43 parts, among them IC2 SPX3819M5-L-3-3_TR, IC3 AT45DB081E-SSHN-B, J1 12401948E412A, J2 Conn_01x02_Pin, J3 Conn_01x13_Pin, Q1 PMOS, U1 ESP32-C6, U2 MCP73831-2-OT, Y1 ECS-400-10-37B-CKY-TR3

Commit message: Tidying up
Parts:
- removed J3: Conn_01x13_Pin, 13 pin:SAMTEC_TSM-113-02-T-SV-A, symbol Connector:Conn_01x13_Pin
- added C18, C19: 3p3, 10 uF:CAPC1608X90N, symbol Device:C
- added J4: SAMTEC-FTS-107-03-X-D, SAMTEC-FTS-107-03-X-D, symbol FTS-107-03-L-D:SAMTEC-FTS-107-03-X-D
- added L2: 2n2, 2 nH:MLG0603, symbol Device:L
Connections:
- net ANT: now also C19.2, L2.1; no longer U1.1 (ANT)
- net D/C: now also J4.7
- net FSPICLK: now also J4.5
- net FSPICS5: now also J4.6
- net FSPID: now also J4.4
- net FSPIQ: now also J4.3
- net GND: now also J4.2
- net GNDREF: now also C18.1, C19.1
- net I2CEXT0_SCL_in: now also J4.10
- net I2CEXT0_SDA_in: now also J4.11
- net LCD_BL: now also J4.9
- net LCD_RST: now also J4.8
- net TP_INT: now also J4.12
- net TP_RST: now also J4.13
- net U0RXD: no longer names the net of U1.30 (U0RXD/GPIO17/FSPICS1)
- net U0TXD renamed FSPICS0
- new net: C18.2, L2.2, U1.1 (ANT)
- no-connect marks 15 -> 14

Commit message: updated layout 8/06/2023
Parts:
- removed IC2: SPX3819M5-L-3-3_TR, SOT95P280X145-5N:SOT95P280X145-5N, symbol SOT95P280X145-5N:SPX3819M5-L-3-3_TR
- removed Y1: ECS-400-10-37B-CKY-TR3, ECS4001037BCKYTR3:ECS4001037BCKYTR3, symbol Crystal Oscillator:ECS-400-10-37B-CKY-TR3
- added IC1: SPX3819M5-L-3-3_TR, SOT95P280X145-5N:SOT95P280X145-5N, symbol SPX3819M5-L-3-3_TR:SPX3819M5-L-3-3_TR
- added Y2: ECS-400-10-37B-CKY-TR3, ECS4001037BCKYTR3:ECS4001037BCKYTR3, symbol ECS4001037BCKYTR3:ECS-400-10-37B-CKY-TR3
- C18, C19: footprint 10 uF:CAPC1608X90N -> 3.3 pF:CAPC1005X55N
- J4: footprint SAMTEC-FTS-107-03-X-D -> FTS-107-03-L-D:SAMTEC-FTS-107-03-X-D
- L2: footprint 2 nH:MLG0603 -> 2.2 nH:INDC2012X103N
- R13, R15, R7, R8, R9: footprint 10K Ohm:RESC1608X55N -> 10K Ohm:RESC3116X65N
Connections:
- net GNDREF is gone; now on net GND: C1.2, C10.2, C11.1, C12.1, C13.1, C14.2, C18.1, C19.1, C2.2, C3.2, C4.2, C5.2, C6.2, C9.2, IC3.7 (GND), R11.1, R13.2
- net +3.3V: now also IC1.5 (VOUT)
- net FSPICS0: now also J4.6
- net GND: now also IC1.2 (GND), Y2.2 (GND_1), Y2.4 (GND_2)
- net VBUS: now also IC1.1 (VIN), IC1.3 (EN)
- net XTAL_N: now also Y2.3 (OUT/IN)
- net VDD_SPI: now reaches C11.2, C12.2, U1.23 (VDD_SPI/GPIO27)
- net VDD_SPI: now also J4.1
- net at C13.2: now also IC1.4 (ADJ/BYP)
- net at C9.1, R1.1: now also Y2.1 (IN/OUT)
- net FSPICS5: no longer names the net of U1.34 (GPIO21/SDIO_DATA1/FSPICS5)
- net FSPICS5: no longer J4.6
- no-connect marks 14 -> 16

Commit message: Added Current Screenshots for a Visual Flair.
Other:
- company: (none) -> Evan Eden
- title: (none) -> Prototype Digital Pocket Watch
Changed lines of the file:
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@@
 (kicad_sch (version 20230121) (generator eeschema)
   (paper "A3")
+  (title_block
+    (title "Prototype Digital Pocket Watch")
+    (company "Evan Eden")
+  )
   (junction (at 247.65 36.83) (diameter 0) (color 0 0 0 0)
   )
