File: mainv2/mainv2.kicad_pcb (KiCad board)
At the start: 4 copper layers, 9.8 x 4.5 mm, 43 parts, among them IC2 SPX3819M5-L-3-3_TR, IC3 AT45DB081E-SSHN-B, J1 12401948E412A, J2 Conn_01x02_Pin, J3 Conn_01x13_Pin, Q1 PMOS, U1 ESP32-C6, U2 MCP73831-2-OT, Y1 ECS-400-10-37B-CKY-TR3

Commit message: Tidying up
Parts:
- removed J3: Conn_01x13_Pin, 13 pin:SAMTEC_TSM-113-02-T-SV-A
- added C**: CAPC1005X55N, 3.3 pF:CAPC1005X55N, F.Cu at (145.7, 72.0)
- added C**: CAPC1005X55N, 3.3 pF:CAPC1005X55N, F.Cu at (151.4, 72.1)
- added J4: SAMTEC-FTS-107-03-X-D, FTS-107-03-L-D:SAMTEC-FTS-107-03-X-D, F.Cu at (135.5, 55.3)
- added L**: INDC2012X103N, 2.2 nH:INDC2012X103N, F.Cu at (148.5, 71.5)
- moved C9 20.5 mm to (149.4, 62.7), turned to -90 degrees
- moved ANT2 16.1 mm to (132.0, 74.5)
- moved Y1 15.5 mm to (145.4, 62.5), turned to 180 degrees
- moved C10 10.9 mm to (141.2, 62.5), turned to 90 degrees
- moved R1 6.93 mm to (148.6, 67.0)
- moved C6 0.08 mm to (154.6, 56.1)
Connections:
- C11 pad 2: Net-(IC3-VCC) -> Net-(U1-VDD_SPI/GPIO27)
- C12 pad 2: Net-(IC3-VCC) -> Net-(U1-VDD_SPI/GPIO27)
- U1 pad 23: Net-(IC3-VCC) -> Net-(U1-VDD_SPI/GPIO27)
- U1 pad 29: /U0TXD -> /FSPICS0
- U1 pad 30: /U0RXD -> unconnected-(U1-U0RXD/GPIO17/FSPICS1-Pad30)
Routing:
- net /FSPICS5: track 40.3 -> 0.00 mm, vias 2 -> 0
- net /FSPICS0: track 0.00 -> 33.0 mm, vias 0 -> 1
- net /ANT: track 9.38 -> 29.2 mm
- net /FSPIQ: track 50.2 -> 31.1 mm
- net Net-(Y1-IN/OUT): track 23.5 -> 10.2 mm
- net Net-(IC3-VCC): track 86.1 -> 74.0 mm
- net GNDREF: track 36.2 -> 24.1 mm, vias 16 -> 15
- net /FSPICLK: track 42.6 -> 30.7 mm
- net /XTAL_N: track 29.8 -> 18.9 mm
- net /TP_INT: track 27.1 -> 36.8 mm, vias 0 -> 1
- net /I2CEXT0_SDA_in: track 30.3 -> 24.0 mm
- net GND: track 41.0 -> 35.8 mm, vias 7 -> 10
- net /LCD_BL: track 32.3 -> 27.2 mm
- net /XTAL_P: track 5.92 -> 10.8 mm
- net /TP_RST: track 22.0 -> 26.9 mm, vias 0 -> 1
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
Commit message: updated layout 8/06/2023
Parts:
- removed C** (x2): CAPC1005X55N, 3.3 pF:CAPC1005X55N
- removed IC2: SPX3819M5-L-3-3_TR, SOT95P280X145-5N:SOT95P280X145-5N
- removed L**: INDC2012X103N, 2.2 nH:INDC2012X103N
- removed Y1: ECS-400-10-37B-CKY-TR3, ECS4001037BCKYTR3:ECS4001037BCKYTR3
- added C18: 3p3, 3.3 pF:CAPC1005X55N, F.Cu at (147.0, 104.1)
- added C19: 3p3, 3.3 pF:CAPC1005X55N, F.Cu at (142.0, 104.2)
- added IC1: SPX3819M5-L-3-3_TR, SOT95P280X145-5N:SOT95P280X145-5N, F.Cu at (156.7, 103.4)
- added L2: 2n2, 2.2 nH:INDC2012X103N, F.Cu at (144.6, 103.7)
- added Y2: ECS-400-10-37B-CKY-TR3, ECS4001037BCKYTR3:ECS4001037BCKYTR3, F.Cu at (144.5, 94.4)
- R13, R15, R7, R8, R9: footprint 10K Ohm:RESC1608X55N -> 10K Ohm:RESC3116X65N
- moved J2 48.6 mm to (141.7, 109.8), turned to 180 degrees
- moved R13 40.7 mm to (167.6, 115.8), turned to 90 degrees
- moved J4 34.5 mm to (134.9, 89.8)
- moved R9 33.2 mm to (149.8, 87.8), turned to 90 degrees
- moved R6 33.0 mm to (154.0, 77.0)
- moved R5 32.9 mm to (154.0, 84.1)
- moved R4 32.9 mm to (154.0, 82.3)
- moved IC3 32.9 mm to (145.9, 80.4)
- moved R3 32.8 mm to (154.0, 80.4)
- moved R2 32.8 mm to (154.0, 78.7)
- moved R8 32.7 mm to (152.6, 87.4), turned to 90 degrees
- moved R7 32.5 mm to (140.8, 80.2)
- moved R1 32.2 mm to (147.5, 99.2)
- moved C9 31.9 mm to (148.2, 94.6)
- moved ANT2 31.8 mm to (133.2, 106.3)
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Connections:
- C1 pad 2: GNDREF -> GND
- C10 pad 2: GNDREF -> GND
- C11 pad 1: GNDREF -> GND
- C11 pad 2: Net-(U1-VDD_SPI/GPIO27) -> /VDD_SPI
- C12 pad 1: GNDREF -> GND
- C12 pad 2: Net-(U1-VDD_SPI/GPIO27) -> /VDD_SPI
- C13 pad 1: GNDREF -> GND
- C14 pad 2: GNDREF -> GND
- C2 pad 2: GNDREF -> GND
- C3 pad 2: GNDREF -> GND
- C4 pad 2: GNDREF -> GND
- C5 pad 2: GNDREF -> GND
- C6 pad 2: GNDREF -> GND
- C9 pad 2: GNDREF -> GND
- IC3 pad 7: GNDREF -> GND
- J4 pad 1: unconnected-(J4-Pad1) -> /VDD_SPI
- R11 pad 1: GNDREF -> GND
- R13 pad 2: GNDREF -> GND
- U1 pad 1: /ANT -> Net-(U1-ANT)
- U1 pad 23: Net-(U1-VDD_SPI/GPIO27) -> /VDD_SPI
- U1 pad 34: /FSPICS5 -> unconnected-(U1-GPIO21/SDIO_DATA1/FSPICS5-Pad34)
Routing:
- net Net-(IC3-VCC): track 74.0 -> 8.54 mm, vias 3 -> 0
- net /VDD_SPI: track 0.00 -> 40.1 mm, vias 0 -> 2
- net GND: track 35.8 -> 69.8 mm, vias 10 -> 16
- net /LCD_RST: track 29.6 -> 54.3 mm
- net GNDREF: track 24.1 -> 0.00 mm, vias 15 -> 0
- net Net-(U1-ANT): track 0.00 -> 21.4 mm
- net /ANT: track 29.2 -> 8.11 mm
- net Net-(J2-Pin_2): track 41.1 -> 27.1 mm, vias 3 -> 0
- net /FSPICS0: track 33.0 -> 44.3 mm, vias 1 -> 2
- net /D1-: track 53.9 -> 65.1 mm
- net VBUS: track 120.2 -> 110.3 mm, vias 5 -> 4
- net /D1+: track 57.1 -> 48.5 mm
- net /D/C: track 38.6 -> 32.1 mm, vias 1 -> 2
- net /XTAL_N: track 18.9 -> 25.0 mm
- net /TP_INT: track 36.8 -> 31.0 mm, vias 1 -> 2
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Other:
- board size 9.8 x 4.5 mm -> 57.2 x 53 mm
- board text removed: "3.3V Rail Starts at (C14)"

Commit message: Board Update
Routing:
- net +3.3V: track 109.1 -> 110.6 mm
- net /I2CEXT0_SCL_in: track 32.7 -> 33.7 mm
- net Net-(C1-Pad1): track 3.17 -> 3.94 mm
